Commit message: Modified parameters for performance

File: urdf/fra2mo_base_macro.xacro (robot description, xacro)
@@ -10,5 +10,5 @@
     <xacro:property name="wheel_mass" value="2.5" />
     <xacro:property name="wheel_radius" value="0.035" />
-    <xacro:property name="wheel_axle" value="0.130" />
+    <xacro:property name="wheel_axle" value="0.124" />
     <!-- Actual body/chassis of the robot -->
     <link name="base_footprint">

Commit message: Fixed expore config file

File: urdf/fra2mo_base_macro.xacro (robot description, xacro)
@@ -10,5 +10,5 @@
     <xacro:property name="wheel_mass" value="2.5" />
     <xacro:property name="wheel_radius" value="0.035" />
-    <xacro:property name="wheel_axle" value="0.124" />
+    <xacro:property name="wheel_axle" value="0.13" />
     <!-- Actual body/chassis of the robot -->
     <link name="base_footprint">
