Commit message: Initial commit

File: urdf/fra2mo.urdf.xacro (robot description, xacro)
@@ -1,8 +1,10 @@
 <?xml version="1.0"?>
 <robot xmlns:xacro="http://www.ros.org/wiki/xacro" name="fra2mo" >
-  <xacro:include filename="$(find ros2_fra2mo)/urdf/fra2mo_base_macro.xacro"/>
-  <xacro:include filename="$(find ros2_fra2mo)/urdf/lidar_gazebo_macro.xacro"/>
-  <!-- <xacro:include filename="$(find ros2_fra2mo)/urdf/d435_gazebo_macro.xacro" />  -->
+  <xacro:include filename="$(find fra2mo_armando)/urdf/fra2mo_base_macro.xacro"/>
+  <xacro:include filename="$(find fra2mo_armando)/urdf/lidar_gazebo_macro.xacro"/>
+  <xacro:include filename="$(find fra2mo_armando)/urdf/armando_macro.xacro"/>
+  <!-- <xacro:include filename="$(find fra2mo_armando)/urdf/d435_gazebo_macro.xacro" />  -->
   <xacro:property name="LIDAR" value="True"/>
+  <xacro:property name="ARM" value="True"/>
   <!--<xacro:property name="DEPTH" value="True"/>-->
   <!-- Diff Drive Robot Base -->
@@ -11,4 +13,8 @@
   <xacro:if value="${LIDAR}">
     <xacro:lidar_gazebo_sensor parent="lidar_link"/>
+  </xacro:if>
+  <!-- Armando Manipulator -->
+  <xacro:if value="${ARM}">
+    <xacro:armando parent="top_mount_link" prefix="arm_" origin_xyz="0 0 0.04" origin_rpy="0 0 0"/>
   </xacro:if>
   <!-- RGBD Sensor (D435 Camera) -->

File: urdf/fra2mo_base_macro.xacro (robot description, xacro)
@@ -1,5 +1,5 @@
 <?xml version="1.0"?>
 <robot  xmlns:xacro="http://www.ros.org/wiki/xacro">
-  <xacro:include filename="$(find ros2_fra2mo)/urdf/utility_macro.xacro" />
+  <xacro:include filename="$(find fra2mo_armando)/urdf/utility_macro.xacro" />
   <!-- WHOLE BASE MACRO-->
   <xacro:macro name="fra2mo_base" > <!--fb : front, back ; lr: left, right -->
@@ -11,4 +11,8 @@
     <xacro:property name="wheel_radius" value="0.035" />
     <xacro:property name="wheel_axle" value="0.13" />
+    <xacro:property name="mount_height" value="0.01" />
+    <xacro:property name="mount_radius" value="0.09" />
+    <xacro:property name="mount_mass" value="0.5" />
+    <xacro:property name="mount_offset_z" value="0.18" />
     <!-- Actual body/chassis of the robot -->
     <link name="base_footprint">
@@ -24,5 +28,5 @@
       <visual>
         <geometry>
-          <mesh filename="file://$(find ros2_fra2mo)/meshes/rl_fra2mo_body.stl" scale="0.001 0.001 0.001" />
+          <mesh filename="file://$(find fra2mo_armando)/meshes/rl_fra2mo_body.stl" scale="0.001 0.001 0.001" />
         </geometry>
         <material name="Blue" />
@@ -47,5 +51,5 @@
       <visual>
         <geometry>
-          <mesh filename="file://$(find ros2_fra2mo)/meshes/rl_fra2mo_wheel.stl" scale="0.001 0.001 0.001" />
+          <mesh filename="file://$(find fra2mo_armando)/meshes/rl_fra2mo_wheel.stl" scale="0.001 0.001 0.001" />
         </geometry>
         <material name="Black" />
@@ -54,5 +58,5 @@
       <collision>
         <geometry>
-          <mesh filename="file://$(find ros2_fra2mo)/meshes/rl_fra2mo_wheel.stl" scale="0.001 0.001 0.001" />
+          <mesh filename="file://$(find fra2mo_armando)/meshes/rl_fra2mo_wheel.stl" scale="0.001 0.001 0.001" />
         </geometry>
         <origin xyz="0 0 0" rpy="0 0 0" />
@@ -68,12 +72,12 @@
       <visual>
         <geometry>
-          <mesh filename="file://$(find ros2_fra2mo)/meshes/rl_fra2mo_wheel.stl" scale="0.001 0.001 0.001" />
+          <mesh filename="file://$(find fra2mo_armando)/meshes/rl_fra2mo_wheel.stl" scale="0.001 0.001 0.001" />
         </geometry>
-        <material name="Black"/>
+        <material name="Black" />
         <origin xyz="0 0 0" rpy="0 0 0" />
       </visual>
       <collision>
         <geometry>
-          <mesh filename="file://$(find ros2_fra2mo)/meshes/rl_fra2mo_wheel.stl" scale="0.001 0.001 0.001" />
+          <mesh filename="file://$(find fra2mo_armando)/meshes/rl_fra2mo_wheel.stl" scale="0.001 0.001 0.001" />
         </geometry>
         <origin xyz="0 0 0" rpy="0 0 0" />
@@ -89,4 +93,23 @@
     </link>
     <link name="lidar_link" />
+    <link name="top_mount_link">
+      <visual>
+        <geometry>
+          <cylinder length="${mount_height}" radius="${mount_radius}" />
+        </geometry>
+        <material name="Blue" />
+        <origin xyz="0 0 0" rpy="0 0 0" />
+      </visual>
+      <collision>
+        <geometry>
+          <cylinder length="${mount_height}" radius="${mount_radius}" />
+        </geometry>
+      </collision>
+      <inertial>
+        <origin xyz="0 0 0" />
+        <mass value="${mount_mass}" />
+        <xacro:cylinder_inertia m="${mount_mass}" r="${mount_radius}" h="${mount_height}" />
+      </inertial>
+    </link>
     <!-- Joints -->
     <joint name="base_footprint_joint" type="fixed">
@@ -121,4 +144,9 @@
       <origin xyz="0.0 0.0 0.125" rpy="0 0 0" />
     </joint>
+    <joint name="top_mount_joint" type="fixed">
+      <parent link="base_link" />
+      <child link="top_mount_link" />
+      <origin xyz="0.0 0.0 ${mount_offset_z}" rpy="0 0 0" />
+    </joint>
     <!-- Gazebo Material Assignments
     <gazebo reference="base_link">
@@ -148,5 +176,5 @@
       </actuator>
     </transmission>
-    <!-- Plugin for differential drive control in Gazebo-->
+    <!-- Plugin for differential drive control in Gazebo -->
     <gazebo>
       <plugin name="ignition::gazebo::systems::DiffDrive" filename="libignition-gazebo-diff-drive-system.so">
@@ -155,6 +183,4 @@
         <wheel_separation>${wheel_axle}</wheel_separation>
         <wheel_radius>${wheel_radius}</wheel_radius>
-        <!--<frame_id>base_footprint</frame_id> TO LOOK
-        <ignition_frame_id>base_footprint</ignition_frame_id>-->
         <odom_publish_frequency>50</odom_publish_frequency>
         <topic>cmd_vel</topic>

File: urdf/lidar_gazebo_macro.xacro (robot description, xacro)
@@ -1,5 +1,5 @@
 <?xml version="1.0"?>
 <robot xmlns:xacro="http://www.ros.org/wiki/xacro" name="lidar_gazebo_macro" >
-  <!--<xacro:include filename="$(find ros2_fra2mo)/urdf/utility_macro.xacro" />-->
+  <!-- utility_macro.xacro already included in fra2mo_base_macro.xacro -->
   <xacro:macro name="lidar_gazebo_sensor" params="parent">
     <link name="laser_frame">
@@ -12,5 +12,5 @@
         <origin rpy="0 0 ${-M_PI_2}" xyz="0.0 0.0 -0.031" />
         <geometry>
-          <mesh filename="file://$(find ros2_fra2mo)/meshes/lidar.stl" scale="0.001 0.001 0.001" />
+          <mesh filename="file://$(find fra2mo_armando)/meshes/lidar.stl" scale="0.001 0.001 0.001" />
         </geometry>
         <material name="White" />
@@ -30,5 +30,4 @@
     <gazebo reference="laser_frame">
       <sensor name="laser_frame" type="gpu_lidar">
-          <!--<pose relative_to="laser_frame">0 0 0 0 0 0</pose>--> <!--TO LOOK-->
           <topic>lidar</topic>
           <update_rate>10</update_rate>
@@ -54,6 +53,6 @@
               </range>
             </ray>
-            <always_on>false</always_on>
-            <visualize>false</visualize>
+            <always_on>true</always_on>
+            <visualize>true</visualize>
             <frame_id>laser_frame</frame_id> <!--TO LOOK-->
             <ignition_frame_id>laser_frame</ignition_frame_id>
@@ -67,7 +66,7 @@
     </plugin>
   </gazebo>-->
-  <gazebo>
+  <!--<gazebo>
   <plugin filename="ignition-gazebo-sensors-system" name="gz::sim::systems::Sensors" />
-  </gazebo>
+  </gazebo>-->
   </xacro:macro>
 </robot>
